Commit message: USV integration

File: tum_simulator/cvg_sim_gazebo/urdf/decorations.urdf.xacro (robot description, xacro)
@@ -112,6 +112,5 @@
       <visual>
         <geometry>
-          <!--<box size="10 10 10" />-->
-          <mesh filename="/home/pulver/.gazebo/models/marker/meshes/artag_01.dae" scale="10 10 10"/>
+          <mesh filename="file:///home/pulver/.gazebo/models/marker/meshes/artag_01.dae" scale="10 10 10"/>
         </geometry>
       </visual>

File: tum_simulator/kingfisher_gazebo/urdf/kingfisher_urdf.xacro (robot description, xacro)
@@ -144,5 +144,5 @@
       <geometry>
         <!--<box size="10 10 10" />-->
-        <mesh filename="/home/pulver/.gazebo/models/marker/meshes/artag_01.dae" scale="10 10 10"/>
+        <mesh filename="file:///home/pulver/.gazebo/models/marker/meshes/artag_01.dae" scale="10 10 10"/>
       </geometry>
     </visual>
